File: PCB_Hub/PCB_Hub.kicad_pcb (KiCad board)
At the start: 2 copper layers, 100 x 37.2 mm, 8 parts, among them U1 TSR_1-2433

Commit message: complete artwork
Routing:
- net GND: track 0.00 -> 92.6 mm
- net +5V: track 0.00 -> 52.3 mm
- net 1PPS: track 0.00 -> 28.9 mm
- net Due RX: track 0.00 -> 28.1 mm
- net Due TX: track 0.00 -> 23.6 mm
- net +3V3: track 0.00 -> 22.8 mm
- net Net-(JP1-Pad1): track 0.00 -> 20.9 mm
- added copper zone on B.Cu, net GND
- added copper zone on F.Cu, net GND
Changed lines of the file:
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@@
     (effects (font (size 1 1) (thickness 0.15)))
   )
+  (segment (start 116.055 154.17) (end 114.93 153.045) (width 0.25) (layer "F.Cu") (net 1))
+  (segment (start 135.875 151.145) (end 134.62 151.145) (width 0.25) (layer "F.Cu") (net 1))
+  (segment (start 134.62 131.445) (end 135.255 131.445) (width 0.25) (layer "F.Cu") (net 1))
+  (segment (start 109.855 130.175) (end 109.855 141.605) (width 0.25) (layer "F.Cu") (net 1))
+  (segment (start 137.16 149.86) (end 135.875 151.145) (width 0.25) (layer "F.Cu") (net 1))
+  (segment (start 131.595 154.17) (end 116.055 154.17) (width 0.25) (layer "F.Cu") (net 1))
+  (segment (start 114.93 120.025) (end 111.115 120.025) (width 0.25) (layer "F.Cu") (net 1))
+  (segment (start 137.16 133.35) (end 137.16 149.86) (width 0.25) (layer "F.Cu") (net 1))
+  (segment (start 111.115 120.025) (end 106.68 124.46) (width 0.25) (layer "F.Cu") (net 1))
+  (segment (start 135.255 131.445) (end 137.16 133.35) (width 0.25) (layer "F.Cu") (net 1))
+  (segment (start 106.68 127) (end 109.855 130.175) (width 0.25) (layer "F.Cu") (net 1))
+  (segment (start 106.68 124.46) (end 106.68 127) (width 0.25) (layer "F.Cu") (net 1))
+  (segment (start 134.62 151.145) (end 131.595 154.17) (width 0.25) (layer "F.Cu") (net 1))
+  (segment (start 108.595 153.045) (end 107.95 152.4) (width 0.25) (layer "B.Cu") (net 1))
+  (segment (start 115.57 120.65) (end 114.945 120.025) (width 0.25) (layer "B.Cu") (net 1))
+  (segment (start 107.95 152.4) (end 107.95 143.51) (width 0.25) (layer "B.Cu") (net 1))
+  (segment (start 114.945 120.025) (end 114.93 120.025) (width 0.25) (layer "B.Cu") (net 1))
+  (segment (start 107.95 143.51) (end 109.855 141.605) (width 0.25) (layer "B.Cu") (net 1))
+  (segment (start 114.93 153.045) (end 108.595 153.045) (width 0.25) (layer "B.Cu") (net 1))
+  (segment (start 107.95 143.51) (end 108.545 144.105) (width 0.25) (layer "F.Cu") (net 2))
+  (segment (start 107.95 129.77) (end 107.95 143.51) (width 0.25) (layer "F.Cu") (net 2))
+  (segment (start 116.05 141.76) (end 112.2 141.76) (width 0.25) (layer "F.Cu") (net 2))
+  (segment (start 104.14 125.96) (end 107.95 129.77) (width 0.25) (layer "F.Cu") (net 2))
+  (segment (start 134.62 133.985) (end 131.295 137.31) (width 0.25) (layer "F.Cu") (net 2))
+  (segment (start 112.2 141.76) (end 109.855 144.105) (width 0.25) (layer "F.Cu") (net 2))
+  (segment (start 131.295 138.270991) (end 130.635991 138.93) (width 0.25) (layer "F.Cu") (net 2))
+  (segment (start 104.14 124.46) (end 104.14 125.96) (width 0.25) (layer "F.Cu") (net 2))
+  (segment (start 130.635991 138.93) (end 118.88 138.93) (width 0.25) (layer "F.Cu") (net 2))
+  (segment (start 118.88 138.93) (end 116.05 141.76) (width 0.25) (layer "F.Cu") (net 2))
+  (segment (start 131.295 137.31) (end 131.295 138.270991) (width 0.25) (layer "F.Cu") (net 2))
+  (segment (start 108.545 144.105) (end 109.855 144.105) (width 0.25) (layer "F.Cu") (net 2))
+  (segment (start 109.855 146.605) (end 111.155 145.305) (width 0.25) (layer "B.Cu") (net 3))
+  (segment (start 111.155 128.875) (end 114.925 125.105) (width 0.25) (layer "B.Cu") (net 3))
+  (segment (start 111.155 145.305) (end 111.155 128.875) (width 0.25) (layer "B.Cu") (net 3))
+  (segment (start 114.925 125.105) (end 114.93 125.105) (width 0.25) (layer "B.Cu") (net 3))
+  (segment (start 121.13 141.76) (end 116.84 146.05) (width 0.25) (layer "F.Cu") (net 4))
+  (segment (start 134.62 139.065) (end 131.925 141.76) (width 0.25) (layer "F.Cu") (net 4))
+  (segment (start 116.05 146.84) (end 112.24 146.84) (width 0.25) (layer "F.Cu") (net 4))
+  (segment (start 116.84 146.05) (end 116.05 146.84) (width 0.25) (layer "F.Cu") (net 4))
+  (segment (start 112.24 146.84) (end 110.49 148.59) (width 0.25) (layer "F.Cu") (net 4))
+  (segment (start 131.925 141.76) (end 121.13 141.76) (width 0.25) (layer "F.Cu") (net 4))
+  (segment (start 121.13 144.3) (end 116.05 149.38) (width 0.25) (layer "F.Cu") (net 5))
+  (segment (start 116.05 149.38) (end 112.08 149.38) (width 0.25) (layer "F.Cu") (net 5))
+  (segment (start 131.925 144.3) (end 121.13 144.3) (width 0.25) (layer "F.Cu") (net 5))
+  (segment (start 112.08 149.38) (end 109.855 151.605) (width 0.25) (layer "F.Cu") (net 5))
+  (segment (start 134.62 141.605) (end 131.925 144.3) (width 0.25) (layer "F.Cu") (net 5))
+  (segment (start 133.365 149.845) (end 134.62 149.845) (width 0.25) (layer "F.Cu") (net 7))
+  (segment (start 114.93 150.505) (end 116.055 151.63) (width 0.25) (layer "F.Cu") (net 7))
+  (segment (start 116.055 151.63) (end 131.58 151.63) (width 0.25) (layer "F.Cu") (net 7))
+  (segment (start 131.58 151.63) (end 133.365 149.845) (width 0.25) (layer "F.Cu") (net 7))
+  (segment (start 109.7 123.98) (end 126.215 123.98) (width 0.25) (layer "F.Cu") (net 8))
+  (segment (start 126.215 123.98) (end 130.17 120.025) (width 0.25) (layer "F.Cu") (net 8))
+  (segment (start 109.22 124.46) (end 109.7 123.98) (width 0.25) (layer "F.Cu") (net 8))
+  (segment (start 130.165 120.025) (end 130.17 120.025) (width 0.25) (layer "B.Cu") (net 8))
+  (zone (net 1) (net_name "GND") (layers F&B.Cu) (hatch edge 0.508)
+    (connect_pads (clearance 0.508))
+    (min_thickness 0.254) (filled_areas_thickness no)
+    (fill yes (thermal_gap 0.508) (thermal_bridge_width 0.508))
+    (polygon
+      (pts
+        (xy 200.66 157.48)
+        (xy 96.52 156.21)
+        (xy 95.25 115.57)
+        (xy 201.93 115.57)
+      )
+    )
+  )
 )
